File: kicad/macpro62-io-risers/riser_hdmi/riser_hdmi.kicad_pcb (KiCad board)
At the start: 4 copper layers, 24.8 x 14.4 mm, 4 parts, among them J1 HDMI HOAUC HYC79-HDMIA19-105 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, J10 DF40C-40DS-0.4V(51) TBC riser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

Commit message: I/O: ports tilted 12.5 deg per stock, riser edge trims, USB-A B2B moved on top, outer-face plug seats, D21-D26 removed
Parts:
- J1: value HDMI HOAUC HYC79-HDMIA19-105 (C711353) (mouth 18.41 above main board top) -> HDMI HOAUC HYC79-HDMIA19-105 (C711353) (mouth 17.46 above main board top)
Other:
- board text added: "riser_hdmi A0 12.5 deg"
- board text removed: "riser_hdmi A0 5.3 deg"
Changed lines of the file:
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@@
 	)
 	(net 0 "")
+	(footprint "MP62_RISER:MP62_Riser_Screw_M2"
+		(layer "F.Cu")
+		(at 89 103)
+		(descr "M2 clearance hole for the printed riser cradle (D-IO14).")
+		(property "Reference" "H1"
+			(at 0 -1 0)
+			(layer "F.Fab")
+			(effects
+				(font
+					(size 0.8 0.8)
+					(thickness 0.12)
+				)
+			)
+		)
+		(property "Value" "M2 to the printed wedge cradle (heat-set insert)"
+			(at 0 1 0)
+			(layer "F.Fab")
+			(effects
+				(font
+					(size 0.6 0.6)
+					(thickness 0.1)
+				)
+			)
+		)
+		(property "Datasheet" ""
+			(at 0 0 0)
+			(layer "F.Fab")
+			(hide yes)
+			(effects
+				(font
+					(size 1.27 1.27)
+					(thickness 0.15)
+				)
+			)
+		)
+		(property "Description" ""
+			(at 0 0 0)
+			(layer "F.Fab")
+			(hide yes)
+			(effects
+				(font
+					(size 1.27 1.27)
+					(thickness 0.15)
+				)
+			)
+		)
+		(attr exclude_from_pos_files exclude_from_bom)
+		(fp_circle
+			(center 0 0)
+			(end 2.15 0)
+			(stroke
+				(width 0.05)
+				(type solid)
+			)
+			(fill no)
+			(layer "F.CrtYd")
+		)
+		(pad "" np_thru_hole circle
+			(at 0 0)
+			(size 2.3 2.3)
+			(drill 2.3)
+			(layers "*.Cu" "*.Mask")
+		)
+		(embedded_fonts no)
+	)
 	(footprint "MP62_RISER:MP62_HDMI_A_Vertical_PLACEHOLDER"
 		(layer "F.Cu")
@@
 			)
 		)
-		(property "Value" "HDMI HOAUC HYC79-HDMIA19-105 (C711353) (mouth 18.41 above main board top)"
+		(property "Value" "HDMI HOAUC HYC79-HDMIA19-105 (C711353) (mouth 17.46 above main board top)"
 			(at 0 1 0)
 			(layer "F.Fab")
@@
 	(footprint "MP62_RISER:MP62_Riser_Screw_M2"
 		(layer "F.Cu")
-		(at 89 103)
+		(at 111 97)
 		(descr "M2 clearance hole for the printed riser cradle (D-IO14).")
-		(property "Reference" "H1"
+		(property "Reference" "H2"
 			(at 0 -1 0)
 			(layer "F.Fab")
@@
 		(embedded_fonts no)
 	)
-	(footprint "MP62_RISER:MP62_Riser_Screw_M2"
-		(layer "F.Cu")
-		(at 111 97)
-		(descr "M2 clearance hole for the printed riser cradle (D-IO14).")
-		(property "Reference" "H2"
-			(at 0 -1 0)
-			(layer "F.Fab")
-			(effects
-				(font
-					(size 0.8 0.8)
-					(thickness 0.12)
-				)
-			)
-		)
-		(property "Value" "M2 to the printed wedge cradle (heat-set insert)"
-			(at 0 1 0)
-			(layer "F.Fab")
-			(effects
-				(font
-					(size 0.6 0.6)
-					(thickness 0.1)
-				)
-			)
-		)
-		(property "Datasheet" ""
-			(at 0 0 0)
-			(layer "F.Fab")
-			(hide yes)
-			(effects
-				(font
-					(size 1.27 1.27)
-					(thickness 0.15)
-				)
-			)
-		)
-		(property "Description" ""
-			(at 0 0 0)
-			(layer "F.Fab")
-			(hide yes)
-			(effects
-				(font
-					(size 1.27 1.27)
-					(thickness 0.15)
-				)
-			)
-		)
-		(attr exclude_from_pos_files exclude_from_bom)
-		(fp_circle
-			(center 0 0)
-			(end 2.15 0)
-			(stroke
-				(width 0.05)
-				(type solid)
-			)
-			(fill no)
-			(layer "F.CrtYd")
-		)
-		(pad "" np_thru_hole circle
-			(at 0 0)
-			(size 2.3 2.3)
-			(drill 2.3)
-			(layers "*.Cu" "*.Mask")
-		)
-		(embedded_fonts no)
-	)
 	(footprint "MP62_RISER:MP62_Hirose_DF40C-40DS-0.4V_PLACEHOLDER"
 		(layer "B.Cu")
@@
 	)
 	(gr_line
-		(start 112.4 107.2)
-		(end 112.4 92.8)
+		(start 87.6 92.8)
+		(end 87.6 107.2)
 		(stroke
 			(width 0.05)
@@
 	)
 	(gr_line
-		(start 87.6 92.8)
-		(end 87.6 107.2)
+		(start 112.4 92.8)
+		(end 87.6 92.8)
 		(stroke
 			(width 0.05)
@@
 	)
 	(gr_line
-		(start 112.4 92.8)
-		(end 87.6 92.8)
+		(start 112.4 107.2)
+		(end 112.4 92.8)
 		(stroke
 			(width 0.05)
@@
 		(layer "Edge.Cuts")
 	)
-	(gr_text "riser_hdmi A0 5.3 deg"
+	(gr_text "riser_hdmi A0 12.5 deg"
 		(at 100 108.7 0)
 		(layer "F.Fab")
