File: kicad/macpro62-backplane/m2_boot.kicad_sch (KiCad schematic)
At the start: 0 parts

Commit message: Cross-board compatibility audit: interface control doc, CR-BP-1 applied, J2/J3 row-swap pinouts, 15-pin face AUX, fan header removed from backplane, CPU board i226/BT1 cleanup
Parts:
- added #BLK7: STUB_M2_BOOT, symbol MP62:STUB_M2_BOOT
Connections:
- net 3V3_BP: now also #BLK7.5 (3V3_BP)
- net SATA0_RX_N: now also #BLK7.4 (SATA0_RX_N)
- net SATA0_RX_P: now also #BLK7.3 (SATA0_RX_P)
- net SATA0_TX_N: now also #BLK7.2 (SATA0_TX_N)
- net SATA0_TX_P: now also #BLK7.1 (SATA0_TX_P)
Other:
- note added: "- SATA0 from the CB Z790 PCH via J1 (SATA-capable HSIO not shared with the M.2 RP9-12 lanes, TBD on the CB)"
- note removed: "- SATA0 from the COM-HPC module via J1 (ccAS has 2 x SATA)"
Changed lines of the file:
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@@
 	(title_block
 		(title "MP62 backplane: OpenCore boot M.2 (SATA)")
-		(date "2026-10-01")
-		(rev "A-bd1")
-		(comment 1 "Block stub: hierarchical labels only, circuit TBD")
+		(date "2026-10-02")
+		(rev "A-bd2")
+		(comment 1 "Block stub: hierarchical labels + one non-BOM stub symbol (#BLKn, passive pins) so ERC sees the nets; circuit TBD")
 	)
 	(hierarchical_label "SATA0_TX_P"
@@
 		(effects (font (size 1.27 1.27)) (justify right))
 	)
+	(symbol
+		(lib_id "MP62:STUB_M2_BOOT")
+		(at 38.1 30.48 0)
+		(unit 1)
+		(exclude_from_sim yes)
+		(in_bom no)
+		(on_board no)
+		(dnp no)
+		(property "Reference" "#BLK7"
+			(at 40.64 27.94 0)
+			(effects (font (size 1.27 1.27)) (justify left) (hide yes))
+		)
+		(property "Value" "STUB_M2_BOOT"
+			(at 40.64 26.67 0)
+			(effects (font (size 1.27 1.27)) (justify left) (hide yes))
+		)
+		(pin "1"
+		)
+		(pin "2"
+		)
+		(pin "3"
+		)
+		(pin "4"
+		)
+		(pin "5"
+		)
+		(instances
+			(project "backplane"
+				(path "/6a1c2d3e-0000-4000-8000-000000000062/b3090511-443b-463a-9e23-87e8afb8be66"
+					(reference "#BLK7")
+					(unit 1)
+				)
+			)
+		)
+	)
 	(text "BLOCK STUB (rev A block diagram). Contents planned:"
 		(exclude_from_sim no)
@@
 		(effects (font (size 1.27 1.27)) (justify left bottom))
 	)
-	(text "- SATA0 from the COM-HPC module via J1 (ccAS has 2 x SATA)"
+	(text "- SATA0 from the CB Z790 PCH via J1 (SATA-capable HSIO not shared with the M.2 RP9-12 lanes, TBD on the CB)"
 		(exclude_from_sim no)
 		(at 76.20 43.18 0)
