File: kicad/macpro62-storage-face/macpro62-storage-face.kicad_sch (KiCad schematic)
At the start: 154 parts, among them J1 MCIO124 RA G97R24332HR, J20 bus-bar lug +12V_IN, J21 bus-bar lug GND, J22 bus-bar lug +12V_IN, J23 bus-bar lug GND, J3 J_AUX SM15B-GHS-TB, J5 M.2 M-key H4.2 LOTES APCI0107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, J6 M.2 M-key H4.2 LOTES APCI0107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, J7 M.2 M-key H4.2 LOTES APCI0107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, J8 M.2 M-key H4.2 LOTES APCI0107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, Q1 N-MOSFET 30V <=5mOhm 5x6, U1 ASM2824 (JLC C9900092023), U10 74LVC2G07, U11 TMP1075DSGR @0x49 (THERM_TRIP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, U12 74LVC2G07, U2 TPS259824ONRGER (C2155766), U3 LM74700-Q1 (DBV), U4 TPS56C215RNNR (C473372), U5 TLV62585DRL VDD_CORE (voltage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, U6 BL24C64A-SFRC @0x50, U7 TMP1075DSGR @0x48 (THERM_ALER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, U8 W25Q16JVSSIQ class (size TBD), U9 74LVC2G07, Y1 25MHz 3225 (populate only if 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

Commit message: ICD rev 2: 45 deg faces, 445 W ceiling + live power target (INA228 telemetry), ribbon MCIO jog cables, BT on S0, fan fail-safe, port-module I2C map
Parts:
- removed C520: 47uF 6.3V 1206 (3V3_SSD), MP62_Storage:C_0402_1005Metric, symbol MP62_Storage:C
- added C520: 47uF 6.3V 1206 (3V3_SSD), MP62_Storage:C_0402_1005Metric, symbol MP62_Storage:C
- added C520: 100nF U13 VS, MP62_Storage:C_0402_1005Metric, symbol MP62_Storage:C
- added R520: 2 mOhm 1% 2512 Kelvin shunt (Face S 12 V, 3.3 A -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, MP62_Storage:R_2512_6332Metric, symbol MP62_Storage:R
- added U13: INA228AIDGSR @0x40 (A0 = A1 = GND) on FACE_SMB; A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, MP62_Storage:VSSOP-10_3x3mm_P0.5mm, symbol MP62_Storage:INA228
Connections:
- net +12V_PROT: now also R520.1, U13.10 (IN+); no longer U2.1 (IN)
- net 3V3_AUX: now also C520.1, U13.6 (VS)
- net 3V3_SSD: now also C520.1
- net FACE_SMB_ALERT#: now also U13.3 (ALERT)
- net FACE_SMB_CLK: now also U13.5 (SCL)
- net FACE_SMB_DAT: now also U13.4 (SDA)
- net GND: now also C520.2, C520.2, U13.1 (A1), U13.2 (A0), U13.7 (GND)
- new net +12V_PROT_S: R520.2, U13.8 (VBUS), U13.9 (IN-), U2.1 (IN)
