File: kicad/macpro62-io-board/macpro62-io-board.kicad_pcb (KiCad board)
At the start: 6 copper layers, 101 x 173.6 mm, 165 parts, among them J1 IOB-HS1 MCIO 124 RA <- CB J3 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, J2 DISPLAY-LINK MCIO 74 RA <- Fa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, J25 ETH1 i226-V #1: ZJLQ-RJ45-SMD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, J26 ETH2 i226-V #2: ZJLQ-RJ45-SMD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, J28 Stock audio module connector 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, J29 Speaker 2P (stock lead; pitch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, J3 Stock PSU DC-out 12P (UNCONFI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, J30 Optional stock/remote power b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, J31 I/O-wall (821-2222) flex ZIF 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, J4 Stock PSU signal 6P (UNCONFIR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, J5 PSU pass-through -> BP J2 (12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, J6 IOB-LINK GH15 <- BP J6, J7 CONN_C fan + AirPort 2x20 @0.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, J8 Fan-assembly antenna coax: U.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, J9 Optional antenna pass-through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, SW1 DNP with the stock 821-2222-A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, SW2 DIAG button, T1 ETH1 2.5G magnetics JASN V24P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, T2 ETH2 2.5G magnetics JASN V24P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, U1 TPS65994AD PD #1 (C1, C2), U11 TUSB1046A C1 alt-mode mux/red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, U12 TUSB1046A C2 alt-mode mux/red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, U13 TUSB1046A C3 alt-mode mux/red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, U14 TUSB1046A C4 alt-mode mux/red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, U15 TUSB1046A C5 alt-mode mux/red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, U16 TUSB1046A C6 alt-mode mux/red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, U2 TPS65994AD PD #2 (C3, C4), U21 TUSB1002A A1 10G redriver, U22 TUSB1002A A2 10G redriver, U23 TUSB1002A A3 10G redriver, U24 TUSB1002A A4 10G redriver, U25 USB-A A1 VBUS switch 1.5 A (S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, U26 USB-A A2 VBUS switch 1.5 A (S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, U27 USB-A A3 VBUS switch 1.5 A (S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, U28 USB-A A4 VBUS switch 1.5 A (S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, U3 TPS65994AD PD #3 (C5, C6), U30 Hall A (DRV5032 class) - posi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, U31 Hall B (DRV5032 class) - posi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, U32 CH334R hub H1b (C4-C6 + codec), U33 CH334R hub H2 (A1-A4) <- IOB-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, U34 CH334R hub H1a (C1-C3 + H1b) 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, U35 CH334R hub H3 on H2 port 4: A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, U4 PD #1 config SPI flash (W25Q8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, U40 TPS259824ON eFuse 12 V in (15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, U41 TPS56C215 5V_C buck (USB-C VB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, U42 TPS56C215 5V_A buck (USB-A VB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, U43 TLV62585 3V3 (3 A) from 5V_SYS, U50 i226-V 2.5GbE (PCIe x1 from H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, U51 i226-V NVM SPI flash (size pe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, U52 i226-V #2 2.5GbE (PCIe x1 fro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, U53 i226-V #2 NVM SPI flash, U6 PD #2 config SPI flash, U60 TDP158 HDMI 2.0 retimer (GPU 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, U61 1V1 LDO (TDP158 core), U7 PD #3 config SPI flash, U70 C-Media CM108B USB audio code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, U71 PAM8302A mono class-D 2.5 W (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, U80 TLC59116 16-ch I2C LED driver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, U81 LIS2DH12 accelerometer (rotat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, U82 BL24C64A IOB ID EEPROM @0x51, U83 TCA9517 I2C buffer (I2C_SYS <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, U84 74LVC1G07 PD_INT -> IOB_INT_N, U90 EMC2101 fan controller @0x4C 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, U91 ASM1182e PCIe Gen2 switch: up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, U95 TCA9548A @0x70: module ID I2C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, U96 TCA9548A @0x71: module ID I2C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, U97 TCA9555 @0x27 on U96 ch3 (pri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, Y1 12 MHz hub crystal, Y2 12 MHz hub crystal, Y3 12 MHz hub crystal, Y4 25 MHz (i226-V), Y5 12 MHz (CM108B), Y6 25 MHz (i226-V #2), Y7 12 MHz hub crystal (H3)

Commit message: USB-C flex module routed (HYCW417, 0 DRC, matched pairs), 3-mil min on flexes, two flex panels, CH334F + ASM1182e QFN-48 footprints
Parts:
- U32: value CH334R hub H1b (C4-C6 + codec) -> CH334F hub H1b (C4-C6 + codec); footprint MP62_IO:MP62_WCH_CH334R_QFN-24_4x4_P0.5_PLACEHOLDER -> MP62_IO:MP62_WCH_CH334F_QFN-24-1EP_4x4_P0.5_EP2.8
- U33: value CH334R hub H2 (A1-A4) <- IOB-LINK USB2 -> CH334F hub H2 (A1-A4) <- IOB-LINK USB2; footprint MP62_IO:MP62_WCH_CH334R_QFN-24_4x4_P0.5_PLACEHOLDER -> MP62_IO:MP62_WCH_CH334F_QFN-24-1EP_4x4_P0.5_EP2.8
- U34: value CH334R hub H1a (C1-C3 + H1b) <- HS1 USB2 -> CH334F hub H1a (C1-C3 + H1b) <- HS1 USB2; footprint MP62_IO:MP62_WCH_CH334R_QFN-24_4x4_P0.5_PLACEHOLDER -> MP62_IO:MP62_WCH_CH334F_QFN-24-1EP_4x4_P0.5_EP2.8
- U35: value CH334R hub H3 on H2 port 4: A4 + Bluetooth USB2 (J7) + 2 spare -> CH334F hub H3 on H2 port 4: A4 + Bluetooth USB2 (J7) + 2 spare; footprint MP62_IO:MP62_WCH_CH334R_QFN-24_4x4_P0.5_PLACEHOLDER -> MP62_IO:MP62_WCH_CH334F_QFN-24-1EP_4x4_P0.5_EP2.8
- U91: footprint MP62_IO:MP62_ASMedia_ASM1182e_QFN-64_9x9_P0.5_PLACEHOLDER -> MP62_IO:MP62_ASMedia_ASM1182e_QFN-48-1EP_7x7_P0.5_EP5.4
Other:
- board text added: "PLACEHOLDER land patterns: all vertical port connectors, stock audio/PSU connectors, TPS65994AD, TUSB1046A, TUSB1002A, TDP158, i226-V (CH334F + ASM1182e: JLCEDA/EasyEDA land patterns 2026-10-04)."
- board text removed: "PLACEHOLDER land patterns: all vertical port connectors, stock audio/PSU connectors, TPS65994AD, TUSB1046A, TUSB1002A, TDP158, i226-V, CH334R."
