File: kicad/macpro62-io-board/macpro62-io-board.kicad_sch (KiCad schematic)
At the start: 454 parts, among them J1 IOB-HS1 MCIO 124 RA <- CB J3, J11 USB-C C1 receptacle vertical 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, J12 USB-C C2 receptacle vertical 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, J13 USB-C C3 receptacle vertical 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, J14 USB-C C4 receptacle vertical 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, J15 USB-C C5 receptacle vertical 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, J16 USB-C C6 receptacle vertical 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, J2 DISPLAY-LINK MCIO 74 RA <- Fa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, J21 USB 3.2 Gen2 Std-A vertical A1, J22 USB 3.2 Gen2 Std-A vertical A2, J23 USB 3.2 Gen2 Std-A vertical A3, J24 USB 3.2 Gen2 Std-A vertical A4, J25 Non-magnetic vertical RJ45 (E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, J26 Non-magnetic vertical RJ45 (E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, J27 HDMI type A vertical, J28 Stock audio module connector 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, J29 Speaker 2P JST SH vertical (s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, J3 Stock PSU DC-out 12P (PROVISI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, J30 OPTIONAL 2P: stock I/O-wall b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, J31 I/O-wall flex ZIF 14P 0.5 (st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, J4 Stock PSU signal 6P (PROVISIO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, J5 Micro-Fit 2x4 -> BP J2 (1-2 1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, J6 IOB-LINK GH15 vertical <- BP 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, J7 CONN_C fan + AirPort (stock p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, Q90 MMBT3904 remote diode (or omi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, SW1 Power button PTS810 on the IO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, SW2 DIAG button TL3342 (back side), T1 JASN V24P05S 2.5G magnetics (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, T2 JASN V24P05S 2.5G magnetics (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, U1 TPS65994AD PD #1 (C1, C2), U11 TUSB1046A-DCI C1 mux/redriver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, U12 TUSB1046A-DCI C2 mux/redriver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, U13 TUSB1046A-DCI C3 mux/redriver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, U14 TUSB1046A-DCI C4 mux/redriver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, U15 TUSB1046A-DCI C5 mux/redriver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, U16 TUSB1046A-DCI C6 mux/redriver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, U2 TPS65994AD PD #2 (C3, C4), U21 TUSB1002A A1 redriver, U22 TUSB1002A A2 redriver, U23 TUSB1002A A3 redriver, U24 TUSB1002A A4 redriver, U25 SY6280AAC / TPS2553 1.5 A swi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, U26 SY6280AAC / TPS2553 1.5 A swi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, U27 SY6280AAC / TPS2553 1.5 A swi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, U28 SY6280AAC / TPS2553 1.5 A swi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, U3 TPS65994AD PD #3 (C5, C6), U30 DRV5032FB (OD, 5 Hz low power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, U31 DRV5032FB (OD, 5 Hz low power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, U32 CH334R H1b <- H1a port 4, U33 CH334R H2 <- IOB-LINK USB2 (B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, U34 CH334R H1a <- HS1 USB2 (CB PC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, U35 CH334R H3 <- H2 port 4 (A4 + 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, U4 W25Q80DV class 8 Mbit (PD #1 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, U40 TPS259824ONRGER eFuse 12 V (I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, U41 TPS56C215RNNR 5V_C buck 12 A, U42 TPS56C215RNNR 5V_A buck 12 A, U43 TLV62585DRL 3V3 3 A from 5V_A, U50 Intel i226-V 2.5GbE #1 (HS1 k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, U51 i226 #1 NVM 2 Mbit+ SPI flash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, U52 Intel i226-V 2.5GbE #2 (HS1 k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, U53 i226 #2 NVM 2 Mbit+ SPI flash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, U6 W25Q80DV class 8 Mbit (PD #2 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, U60 TDP158RSBR HDMI retimer, U61 TLV75511PDBV 1.1 V LDO (TDP15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, U7 W25Q80DV class 8 Mbit (PD #3 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, U70 CM108B USB audio codec (UAC1), U71 PAM8302AAS 2.5 W mono class-D, U80 TLC59116IPWR @0x60 (A3..A0 = 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, U81 LIS2DH12TR @0x18 (optional ro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, U82 BL24C64A-SFRC IOB ID EEPROM @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, U83 TCA9517DGKR I2C buffer: I2C_S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, U84 74LVC1G07 PD_INT_N -> IOB_INT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, U90 EMC2101 fan controller (SMBus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, U91 ASM1182e PCIe Gen2 switch: up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, U92 3V3 WLAN load switch (TPS2291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, Y1 12MHz 3225 +/-20ppm, Y2 12MHz 3225 +/-20ppm, Y3 12MHz 3225 +/-20ppm, Y4 25MHz 3225 +/-30ppm (i226 #1), Y5 12MHz 3225 (CM108B)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

Commit message: I/O: cover scan check (R inner ~102-110), fan antenna U.FL J8, T8 bracket keep-out, BCM94360 12+6 pinout on CONN_C
Parts:
- removed R203: FB bottom, MP62_IO:R_0402_1005Metric, symbol MP62_IO:R
- removed R204: 10k, MP62_IO:R_0402_1005Metric, symbol MP62_IO:R
- added J8: Fan-assembly antenna coax (stock type/position UN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, MP62_IO:MP62_UFL_Hirose_U.FL-R-SMT-1, symbol MP62_IO:UFL
- added J9: Optional antenna pass-through (DNP) - 50 ohm CPW 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, MP62_IO:MP62_UFL_Hirose_U.FL-R-SMT-1, symbol MP62_IO:UFL
- R146: value 10k (radio on; drive from TLC59116/IOB GPIO if wanted) -> 10k DNP (card LED_WLAN# open-drain, unused); now not fitted; now left out of the parts list
- R148: value 10k -> 0R: Bluetooth 3V3 (card P18) from standby so BT can wake in S3; confirm on M-IOC1
- R149: value 0R (3V3_SB alias: confirm the stock rail on M-IOC1) -> 0R DNP alt: BT from S0 3V3; now not fitted; now left out of the parts list
- R150: value 0R DNP (fan-assembly SMBus, if present) -> 1.8k DDC pull-up (sink side); now fitted; now in the parts list
- R151: value 0R DNP -> 1.8k DDC pull-up (sink side); now fitted; now in the parts list
- R152: value 1.8k DDC pull-up (sink side) -> 100k HPD pull-down
- R153: value 1.8k DDC pull-up (sink side) -> 100k
- R154: value 100k HPD pull-down -> 10k (L+R mix into the mono ADC; CM6646 upgrade = stereo line in)
- R155: value 100k -> 10k
- R156: value 10k (L+R mix into the mono ADC; CM6646 upgrade = stereo line in) -> DNP 2.2k (only if the stock line-in jack is a mic/combo); now not fitted; now left out of the parts list
- R157: value 10k -> 100k jack-detect pull-up
- R158: value DNP 2.2k (only if the stock line-in jack is a mic/combo) -> 100k jack-detect pull-up; now fitted; now in the parts list
- R159: value 100k jack-detect pull-up -> 0R (optical TX/RX module supply; 10R if the module wants filtering)
- R160: value 100k jack-detect pull-up -> DNP: optical input not supported by CM108B (CM6646 upgrade); now not fitted; now left out of the parts list
- R161: value 0R (optical TX/RX module supply; 10R if the module wants filtering) -> 100k (amp off until codec GPIO3 enables; firmware mutes on JD_HP)
- R162: value DNP: optical input not supported by CM108B (CM6646 upgrade) -> DNP 0R (only if J4 5/6 prove to be 3.3 V SMBus)
- R163: value 100k (amp off until codec GPIO3 enables; firmware mutes on JD_HP) -> DNP 0R; now not fitted; now left out of the parts list
- R164: value DNP 0R (only if J4 5/6 prove to be 3.3 V SMBus) -> DNP 0R: GND? (probe)
- R165: value DNP 0R -> DNP 0R: GND? (probe)
- R166: value DNP 0R: GND? (probe) -> 0R: community claim pins 3+6 = power button; now fitted; now in the parts list
- R167: value DNP 0R: GND? (probe) -> DNP 0R: LED-MCU logic 3V3? (probe)
- R168: value 0R: community claim pins 3+6 = power button -> DNP 0R: 3V3? (probe); now not fitted; now left out of the parts list
- R169: value DNP 0R: LED-MCU logic 3V3? (probe) -> 0R: button return (pins 3+6); now fitted; now in the parts list
- R170: value DNP 0R: 3V3? (probe) -> DNP 0R: LED-MCU I2C SCL? (probe; must be 3.3 V)
- R171: value 0R: button return (pins 3+6) -> DNP 0R: LED-MCU I2C SDA? (probe); now not fitted; now left out of the parts list
- R172: value DNP 0R: LED-MCU I2C SCL? (probe; must be 3.3 V) -> DNP 0R: flex IRQ/motion? (probe)
- R173: value DNP 0R: LED-MCU I2C SDA? (probe) -> DNP 0R: LED supply 5 V? (probe; S0 only)
- R174: value DNP 0R: flex IRQ/motion? (probe) -> DNP 0R: GND? (probe)
- R175: value DNP 0R: LED supply 5 V? (probe; S0 only) -> DNP 0R: 3V3? (probe)
- R177: value DNP 0R: 3V3? (probe) -> DNP 0R: GND? (probe)
- R178: value DNP 0R: GND? (probe) -> 10k (read via PD #1 GPIO2; S0 only); now fitted; now in the parts list
- R179: value DNP 0R: GND? (probe) -> REXT ~ 2.7k (Iout ~ 7 mA max; PWM per channel); now fitted; now in the parts list
- R180: value 10k (read via PD #1 GPIO2; S0 only) -> 10k (write-protect by default)
- R181: value REXT ~ 2.7k (Iout ~ 7 mA max; PWM per channel) -> DNP 0R (program); now not fitted; now left out of the parts list
- R182: value 10k (write-protect by default) -> 4.7k
- R183: value DNP 0R (program) -> 4.7k; now fitted; now in the parts list
- R184: value 4.7k -> 10k (DNP if the BP pulls up); now not fitted; now left out of the parts list
- R185: value 4.7k -> UVLO top (~10.5 V on)
- R186: value 10k (DNP if the BP pulls up) -> UVLO bottom; now fitted; now in the parts list
- R187: value UVLO top (~10.5 V on) -> ILIM ~10 A (value per datasheet)
- R188: value UVLO bottom -> IMON (value per datasheet)
- R189: value ILIM ~10 A (value per datasheet) -> 10k
- R190: value IMON (value per datasheet) -> 10k
- R191: value 10k -> 0R (fault -> IOB_INT_N, OD)
- R192: value 10k -> MODE strap (FCCM, 800 kHz)
- R193: value 0R (fault -> IOB_INT_N, OD) -> FB top (5.10 V)
- R194, R198: value MODE strap (FCCM, 800 kHz) -> FB bottom
- R195, R199: value FB top (5.10 V) -> 10k PG pull-up
- R196: value FB bottom -> MODE strap (FCCM, 800 kHz)
- R197: value 10k PG pull-up -> FB top (5.10 V)
- R200: value FB bottom -> FB top (3.3 V)
- R201: value 10k PG pull-up -> FB bottom
- R202: value FB top (3.3 V) -> 10k
Connections:
- net +12V_MAIN: now also R185.1; no longer R187.1
- net 3V3: now also R159.1, R175.2, R178.2, R182.2, R183.2, R200.1; no longer R146.2, R148.2, R161.1, R177.2, R180.2, R184.2, R185.2, R202.1
- net 3V3_SB: now also R148.2, R167.2, R168.2, R180.2, R184.2, R189.2, R190.2, R195.2, R199.2, R202.2; no longer J7.34 (3V3_SB), R149.1, R169.2, R170.2, R182.2, R186.2, R191.2, R192.2, R197.2, R201.2
- net 3V3_WL: now also R146.2
- net 5V_A: now also R173.2, R197.1; no longer R175.2, R199.1
- net 5V_C: now also R193.1; no longer R195.1
- net AMP_SD#: now also R161.1; no longer R163.1
- net AUD_3V3: now also R157.2, R158.2; no longer R159.2, R160.2
- net AUD_OPT_3V3: now also R159.2; no longer R161.2
- net BK3_FB: now also R200.2, R201.1; no longer R202.2
- net BKA_FB: now also R197.2, R198.1; no longer R199.2, R200.1
- net BKA_MODE: now also R196.1; no longer R198.1
- net BKC_FB: now also R193.2, R194.1; no longer R195.2, R196.1
- net BKC_MODE: now also R192.1; no longer R194.1
- net DIAG_BTN_N: now also R178.1; no longer R180.1
- net DL_HPD2: now also R153.1; no longer R155.1
- net EFUSE_EN: now also R185.2, R186.1; no longer R187.2, R188.1
- net EFUSE_FLT#: now also R190.1, R191.1; no longer R192.1, R193.1
- net EFUSE_ILIM: now also R187.1; no longer R189.1
- net EFUSE_IMON: now also R188.1; no longer R190.1
- net EFUSE_PG: now also R189.1; no longer R191.1
- net GND: now also R152.2, R153.2, R160.2, R161.2, R164.2, R165.2, R169.2, R174.2, R177.2, R186.2, R187.2, R192.2, R201.2, J8.2 (GND), J9.2 (GND); no longer R154.2, R155.2, R162.2, R163.2, R166.2, R167.2, R171.2, R178.2, R183.2, R189.2, R190.2, R200.2
- net HDMI_5V_OUT: now also R150.2, R151.2; no longer R152.2, R153.2
- net HDMI_HPD: now also R152.1; no longer R154.1
- net HDMI_SCL: now also R150.1; no longer R152.1
- net HDMI_SDA: now also R151.1; no longer R153.1
- net I2C_PD_SCL: now also R182.1; no longer R184.1
- net I2C_PD_SDA: now also R183.1; no longer R185.1
- net I2C_SYS_SCL: now also R162.2, R170.2; no longer R150.2, R164.2, R172.2
- net I2C_SYS_SDA: now also R163.2, R171.2; no longer R151.2, R165.2, R173.2
- net IOB_EE_WP: now also R180.1, R181.1; no longer R182.1, R183.1
- net IOB_INT_N: now also R172.2, R184.1, R191.2; no longer R174.2, R186.1, R193.2
- net JD_HP: now also R157.1; no longer R159.1
- net JD_LINE: now also R158.1; no longer R160.1
- net LED_REXT: now also R179.1; no longer R181.1
- net LINE_IN_MONO: now also R154.2, R155.2; no longer R157.2, R158.2
- net LINE_L: now also R154.1; no longer R156.1
- net LINE_R: now also R155.1; no longer R157.1
- net MIC_BIAS: now also R156.1; no longer R158.1
- net PG_3V3: now also R202.1
- net PG_5VA: now also R199.1; no longer R201.1
- net PG_5VC: now also R195.1; no longer R197.1
- net PSU_SMB_CLK: now also R162.1; no longer R164.1
- net PSU_SMB_DAT: now also R163.1; no longer R165.1
- net PWRBTN_IN_N: now also R166.2; no longer R168.2
- net SPDIF_RX: now also R160.1; no longer R162.1
- net WALL_P1: now also R164.1; no longer R166.1
- net WALL_P10: now also R173.1; no longer R175.1
- net WALL_P11: now also R174.1; no longer R176.1
- net WALL_P12: now also R175.1; no longer R177.1
- net WALL_P13: now also R176.1; no longer R178.1
- net WALL_P14: now also R177.1; no longer R179.1
- net WALL_P2: now also R165.1; no longer R167.1
- net WALL_P3: now also R166.1; no longer R168.1
- net WALL_P4: now also R167.1; no longer R169.1
- net WALL_P5: now also R168.1; no longer R170.1
- net WALL_P6: now also R169.1; no longer R171.1
- net WALL_P7: now also R170.1; no longer R172.1
- net WALL_P8: now also R171.1; no longer R173.1
- net WALL_P9: now also R172.1; no longer R174.1
- net WL_CLKREQ#: now also R147.1; no longer R148.1
- net BT_DISABLE#: no longer names the net of J7.29 (NC29)
- net BT_DISABLE#: no longer R147.1
- net SMB_SCL: no longer names the net of J7.31 (NC31)
- net SMB_SCL: no longer R150.1
- net SMB_SDA: no longer names the net of J7.33 (NC33)
- net SMB_SDA: no longer R151.1
- net W_DISABLE# renamed LED_WLAN#
- new net 3V3_BT: J7.34 (3V3_BT), R148.1, R149.1
- new net RF_ANT_FAN: J8.1 (SIG), J9.1 (SIG)
- no-connect marks 104 -> 107

Commit message: I/O: ports tilted 12.5 deg per stock, riser edge trims, USB-A B2B moved on top, outer-face plug seats, D21-D26 removed
Parts:
- removed D21, D22, D23, D24, D25, D26: DNP (2026-10-02: port lighting via the 821-2222 f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, MP62_IO:LED_0603_1608Metric, symbol MP62_IO:LED
Connections:
- net LEDP1_K: no longer names the net of U80.20 (OUT9)
- net LEDP2_K: no longer names the net of U80.21 (OUT10)
- net LEDP3_K: no longer names the net of U80.22 (OUT11)
- net LEDP4_K: no longer names the net of U80.23 (OUT12)
- net LEDP5_K: no longer names the net of U80.24 (OUT13)
- net LEDP6_K: no longer names the net of U80.25 (OUT14)
- no-connect marks 107 -> 113

Commit message: I/O: ports soldered on flex modules (no rigid PCB), DF40 50-pin standard port-module pinout with ID EEPROM, PA12 cradles + clamp plates, port axes square to plate (12.5 deg variant kept)
Parts:
- removed J11: USB-C C1 receptacle vertical (DL0), MP62_IO:MP62_USB_C_24P_Vertical_PLACEHOLDER, symbol MP62_IO:USB_C_24P
- removed J12: USB-C C2 receptacle vertical (DL1), MP62_IO:MP62_USB_C_24P_Vertical_PLACEHOLDER, symbol MP62_IO:USB_C_24P
- removed J13: USB-C C3 receptacle vertical (DL3), MP62_IO:MP62_USB_C_24P_Vertical_PLACEHOLDER, symbol MP62_IO:USB_C_24P
- removed J14: USB-C C4 receptacle vertical (DL4), MP62_IO:MP62_USB_C_24P_Vertical_PLACEHOLDER, symbol MP62_IO:USB_C_24P
- removed J15: USB-C C5 receptacle vertical (DDIB), MP62_IO:MP62_USB_C_24P_Vertical_PLACEHOLDER, symbol MP62_IO:USB_C_24P
- removed J16: USB-C C6 receptacle vertical (DDIC), MP62_IO:MP62_USB_C_24P_Vertical_PLACEHOLDER, symbol MP62_IO:USB_C_24P
- removed J21: USB 3.2 Gen2 Std-A vertical A1, MP62_IO:MP62_USB_A3_9P_Vertical_PLACEHOLDER, symbol MP62_IO:USB_A3
- removed J22: USB 3.2 Gen2 Std-A vertical A2, MP62_IO:MP62_USB_A3_9P_Vertical_PLACEHOLDER, symbol MP62_IO:USB_A3
- removed J23: USB 3.2 Gen2 Std-A vertical A3, MP62_IO:MP62_USB_A3_9P_Vertical_PLACEHOLDER, symbol MP62_IO:USB_A3
- removed J24: USB 3.2 Gen2 Std-A vertical A4, MP62_IO:MP62_USB_A3_9P_Vertical_PLACEHOLDER, symbol MP62_IO:USB_A3
- removed J27: HDMI type A vertical, MP62_IO:MP62_HDMI_A_Vertical_PLACEHOLDER, symbol MP62_IO:HDMI_A
- added C317: 22uF 0805, MP62_IO:C_0402_1005Metric, symbol MP62_IO:C
- added C318: 10uF 0805, MP62_IO:C_0402_1005Metric, symbol MP62_IO:C
- added C319: 10uF 0402, MP62_IO:C_0402_1005Metric, symbol MP62_IO:C
- added JM1: PMI-50 slot C1: MOD-C USB-C (DL0) - DF40C-50DS-0.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, MP62_IO:MP62_Hirose_DF40C-50DS-0.4V_PLACEHOLDER, symbol MP62_IO:PMI50
- added JM10: PMI-50 slot A4: MOD-A USB-A 10G - DF40C-50DS-0.4V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, MP62_IO:MP62_Hirose_DF40C-50DS-0.4V_PLACEHOLDER, symbol MP62_IO:PMI50
- added JM11: PMI-50 slot HDMI: MOD-H HDMI-A (CEC/UTIL NC) - DF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, MP62_IO:MP62_Hirose_DF40C-50DS-0.4V_PLACEHOLDER, symbol MP62_IO:PMI50
- added JM2: PMI-50 slot C2: MOD-C USB-C (DL1) - DF40C-50DS-0.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, MP62_IO:MP62_Hirose_DF40C-50DS-0.4V_PLACEHOLDER, symbol MP62_IO:PMI50
- added JM3: PMI-50 slot C3: MOD-C USB-C (DL3) - DF40C-50DS-0.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, MP62_IO:MP62_Hirose_DF40C-50DS-0.4V_PLACEHOLDER, symbol MP62_IO:PMI50
- added JM4: PMI-50 slot C4: MOD-C USB-C (DL4) - DF40C-50DS-0.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, MP62_IO:MP62_Hirose_DF40C-50DS-0.4V_PLACEHOLDER, symbol MP62_IO:PMI50
- added JM5: PMI-50 slot C5: MOD-C USB-C (DDIB) - DF40C-50DS-0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, MP62_IO:MP62_Hirose_DF40C-50DS-0.4V_PLACEHOLDER, symbol MP62_IO:PMI50
- added JM6: PMI-50 slot C6: MOD-C USB-C (DDIC) - DF40C-50DS-0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, MP62_IO:MP62_Hirose_DF40C-50DS-0.4V_PLACEHOLDER, symbol MP62_IO:PMI50
- added JM7: PMI-50 slot A1: MOD-A USB-A 10G - DF40C-50DS-0.4V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, MP62_IO:MP62_Hirose_DF40C-50DS-0.4V_PLACEHOLDER, symbol MP62_IO:PMI50
- added JM8: PMI-50 slot A2: MOD-A USB-A 10G - DF40C-50DS-0.4V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, MP62_IO:MP62_Hirose_DF40C-50DS-0.4V_PLACEHOLDER, symbol MP62_IO:PMI50
- added JM9: PMI-50 slot A3: MOD-A USB-A 10G - DF40C-50DS-0.4V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, MP62_IO:MP62_Hirose_DF40C-50DS-0.4V_PLACEHOLDER, symbol MP62_IO:PMI50
- added R203: REXT ~ 2.7k (Iout ~ 7 mA max; PWM per channel), MP62_IO:R_0402_1005Metric, symbol MP62_IO:R
- added R204: 10k (write-protect by default), MP62_IO:R_0402_1005Metric, symbol MP62_IO:R
- added R205: DNP 0R (program), MP62_IO:R_0402_1005Metric, symbol MP62_IO:R
- added R206, R207: 4.7k, MP62_IO:R_0402_1005Metric, symbol MP62_IO:R
- added R208: 10k (DNP if the BP pulls up), MP62_IO:R_0402_1005Metric, symbol MP62_IO:R
- added R209: UVLO top (~10.5 V on), MP62_IO:R_0402_1005Metric, symbol MP62_IO:R
- added R210: UVLO bottom, MP62_IO:R_0402_1005Metric, symbol MP62_IO:R
- added R211: ILIM ~10 A (value per datasheet), MP62_IO:R_0402_1005Metric, symbol MP62_IO:R
- added R212: IMON (value per datasheet), MP62_IO:R_0402_1005Metric, symbol MP62_IO:R
- added R213, R214, R226: 10k, MP62_IO:R_0402_1005Metric, symbol MP62_IO:R
- added R215: 0R (fault -> IOB_INT_N, OD), MP62_IO:R_0402_1005Metric, symbol MP62_IO:R
- added R216, R220: MODE strap (FCCM, 800 kHz), MP62_IO:R_0402_1005Metric, symbol MP62_IO:R
- added R217, R221: FB top (5.10 V), MP62_IO:R_0402_1005Metric, symbol MP62_IO:R
- added R218, R222, R225: FB bottom, MP62_IO:R_0402_1005Metric, symbol MP62_IO:R
- added R219, R223: 10k PG pull-up, MP62_IO:R_0402_1005Metric, symbol MP62_IO:R
- added R224: FB top (3.3 V), MP62_IO:R_0402_1005Metric, symbol MP62_IO:R
- added U95: TCA9548APWR @0x70: ch0-5 C1-C6, ch6-7 A1-A2, MP62_IO:TSSOP-24_4.4x7.8mm_P0.65mm, symbol MP62_IO:TCA9548A
- added U96: TCA9548APWR @0x71: ch0-1 A3-A4, ch2 HDMI, ch3 U97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, MP62_IO:TSSOP-24_4.4x7.8mm_P0.65mm, symbol MP62_IO:TCA9548A
- added U97: TCA9555PWR @0x27 on U96 ch3 (private; not on I2C_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, MP62_IO:TSSOP-24_4.4x7.8mm_P0.65mm, symbol MP62_IO:TCA9555
- C277, C288: value 10uF 0402 -> 100nF
- C282: value 22pF -> 100nF
- C283: value 22pF -> 10uF 0402
- C284: value 4.7uF -> 100nF
- C285: value 100nF -> 22pF
- C286: value 10uF 0402 -> 22pF
- C287: value 100nF -> 4.7uF
- C290: value 100nF (L into IN+) -> 100nF
- C291: value 100nF (R into IN+, mono sum) -> 10uF 0402
- C292: value 220nF (IN- to AGND) -> 10uF 0402
- C293: value 10uF 0603 -> 100nF (L into IN+)
- C294: value 1uF -> 100nF (R into IN+, mono sum)
- C295: value 10uF 1206 25V (header) -> 220nF (IN- to AGND)
- C296: value 100nF (debounce; pull-up on BP) -> 10uF 0603
- C297, C302: value 100nF -> 1uF
- C298: value 100nF -> 10uF 1206 25V (header)
- C299: value 1uF -> 100nF (debounce; pull-up on BP)
- C305: value 100nF (CB keeps 1uF + 0.1uF + diode-OR with 3V3_DSW) -> 100nF
- C306: value dVdt (inrush <= 2 A, value per datasheet) -> 100nF
- C307: value 100nF BOOT -> 100nF
- C308: value 4.7uF VREG5 -> 100nF (CB keeps 1uF + 0.1uF + diode-OR with 3V3_DSW)
- C309: value SS (value per datasheet) -> dVdt (inrush <= 2 A, value per datasheet)
- C313: value 22uF 0805 -> 100nF BOOT
- C314: value 22uF 0805 -> 4.7uF VREG5
- C315: value 10uF 0805 -> SS (value per datasheet)
- C316: value 10uF 0402 -> 22uF 0805
- R150, R151: value 1.8k DDC pull-up (sink side) -> 4.7k
- R152: value 100k HPD pull-down -> 4.7k
- R153: value 100k -> 4.7k
- R154: value 10k (L+R mix into the mono ADC; CM6646 upgrade = stereo line in) -> 4.7k
- R155: value 10k -> 4.7k
- R156: value DNP 2.2k (only if the stock line-in jack is a mic/combo) -> 4.7k; now fitted; now in the parts list
- R157, R158: value 100k jack-detect pull-up -> 4.7k
- R159: value 0R (optical TX/RX module supply; 10R if the module wants filtering) -> 4.7k
- R160: value DNP: optical input not supported by CM108B (CM6646 upgrade) -> 4.7k; now fitted; now in the parts list
- R161: value 100k (amp off until codec GPIO3 enables; firmware mutes on JD_HP) -> 4.7k
- R162: value DNP 0R (only if J4 5/6 prove to be 3.3 V SMBus) -> 4.7k; now fitted; now in the parts list
- R163: value DNP 0R -> 4.7k; now fitted; now in the parts list
- R164, R165: value DNP 0R: GND? (probe) -> 4.7k; now fitted; now in the parts list
- R166: value 0R: community claim pins 3+6 = power button -> 4.7k
- R167: value DNP 0R: LED-MCU logic 3V3? (probe) -> 4.7k; now fitted; now in the parts list
- R168: value DNP 0R: 3V3? (probe) -> 4.7k; now fitted; now in the parts list
- R169: value 0R: button return (pins 3+6) -> 4.7k
- R170: value DNP 0R: LED-MCU I2C SCL? (probe; must be 3.3 V) -> 4.7k; now fitted; now in the parts list
- R171: value DNP 0R: LED-MCU I2C SDA? (probe) -> 4.7k; now fitted; now in the parts list
- R172: value DNP 0R: flex IRQ/motion? (probe) -> 4.7k; now fitted; now in the parts list
- R173: value DNP 0R: LED supply 5 V? (probe; S0 only) -> 4.7k; now fitted; now in the parts list
- R174: value DNP 0R: GND? (probe) -> 1.8k DDC pull-up (sink side); now fitted; now in the parts list
- R175: value DNP 0R: 3V3? (probe) -> 1.8k DDC pull-up (sink side); now fitted; now in the parts list
- R176: value DNP 0R: GND? (probe) -> 100k HPD pull-down; now fitted; now in the parts list
- R177: value DNP 0R: GND? (probe) -> 100k; now fitted; now in the parts list
- R178: value 10k (read via PD #1 GPIO2; S0 only) -> 10k (L+R mix into the mono ADC; CM6646 upgrade = stereo line in)
- R179: value REXT ~ 2.7k (Iout ~ 7 mA max; PWM per channel) -> 10k
- R180: value 10k (write-protect by default) -> DNP 2.2k (only if the stock line-in jack is a mic/combo); now not fitted; now left out of the parts list
- R181: value DNP 0R (program) -> 100k jack-detect pull-up; now fitted; now in the parts list
- R182: value 4.7k -> 100k jack-detect pull-up
- R183: value 4.7k -> 0R (optical TX/RX module supply; 10R if the module wants filtering)
- R184: value 10k (DNP if the BP pulls up) -> DNP: optical input not supported by CM108B (CM6646 upgrade)
- R185: value UVLO top (~10.5 V on) -> 100k (amp off until codec GPIO3 enables; firmware mutes on JD_HP)
- R186: value UVLO bottom -> DNP 0R (only if J4 5/6 prove to be 3.3 V SMBus); now not fitted; now left out of the parts list
- R187: value ILIM ~10 A (value per datasheet) -> DNP 0R; now not fitted; now left out of the parts list
- R188: value IMON (value per datasheet) -> DNP 0R: GND? (probe); now not fitted; now left out of the parts list
- R189: value 10k -> DNP 0R: GND? (probe); now not fitted; now left out of the parts list
- R190: value 10k -> 0R: community claim pins 3+6 = power button
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Connections:
- net +12V_MAIN: now also C298.1, R209.1; no longer C295.1, R185.1
- net 1V1_HDMI: now also C280.1, C281.1, C282.1; no longer C277.1, C278.1, C279.1
- net 3V3: now also C277.1, C278.1, C279.1, C283.1, C284.1, C307.1, C316.1, R150.2, R151.2, R152.2, R153.2, R154.2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; no longer C280.1, C281.1, C304.1, C313.1, C314.1, R159.1, R175.2, R178.2, R182.2, R183.2, R200.1
- net 3V3_SB: now also C304.1, C305.1, C306.1, R191.2, R192.2, C319.1, R204.2, R208.2, R213.2, R214.2, R219.2, R223.2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; no longer C297.1, C298.1, C299.1, C316.1, R167.2, R168.2, R180.2, R184.2, R189.2, R190.2, R195.2, R199.2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
- net 5V_A: now also C291.1, C296.1, C297.1, R197.2, C318.1, R221.1; no longer C288.1, C293.1, C294.1, C315.1, R173.2, R197.1
- net 5V_C: now also R217.1; no longer R193.1
- net A1_SS_RX_N: now also JM7.25 (HS1_N)
- net A1_SS_RX_P: now also JM7.23 (HS1_P)
- net A1_SS_TX_N: now also JM7.19 (HS0_N)
- net A1_SS_TX_P: now also JM7.17 (HS0_P)
- net A1_USB2_DN: now also JM7.31 (USB2_DN)
- net A1_USB2_DP: now also JM7.29 (USB2_DP)
- net A2_SS_RX_N: now also JM8.25 (HS1_N)
- net A2_SS_RX_P: now also JM8.23 (HS1_P)
- net A2_SS_TX_N: now also JM8.19 (HS0_N)
- net A2_SS_TX_P: now also JM8.17 (HS0_P)
- net A2_USB2_DN: now also JM8.31 (USB2_DN)
- net A2_USB2_DP: now also JM8.29 (USB2_DP)
- net A3_SS_RX_N: now also JM9.25 (HS1_N)
- net A3_SS_RX_P: now also JM9.23 (HS1_P)
- net A3_SS_TX_N: now also JM9.19 (HS0_N)
- net A3_SS_TX_P: now also JM9.17 (HS0_P)
- net A3_USB2_DN: now also JM9.31 (USB2_DN)
- net A3_USB2_DP: now also JM9.29 (USB2_DP)
- net A4_SS_RX_N: now also JM10.25 (HS1_N)
- net A4_SS_RX_P: now also JM10.23 (HS1_P)
- net A4_SS_TX_N: now also JM10.19 (HS0_N)
- net A4_SS_TX_P: now also JM10.17 (HS0_P)
- net A4_USB2_DN: now also JM10.31 (USB2_DN)
- net A4_USB2_DP: now also JM10.29 (USB2_DP)
- net AGND: now also C295.2; no longer C292.2
- net AMP_INN: now also C295.1; no longer C292.1
- net AMP_INP: now also C293.2, C294.2; no longer C290.2, C291.2
- net AMP_SD#: now also R185.1; no longer R161.1
- net AUD_3V3: now also C287.1, C288.1, R181.2, R182.2; no longer C284.1, C285.1, R157.2, R158.2
- net AUD_AVDD: now also C289.1, C290.1; no longer C286.1, C287.1
- net AUD_OPT_3V3: now also C292.1, R183.2; no longer C289.1, R159.2
- net AUD_XI: now also C285.1; no longer C282.1
- net AUD_XO: now also C286.1; no longer C283.1
- net BK3_FB: now also R224.2, R225.1; no longer R200.2, R201.1
- net BKA_BOOT: now also C313.1; no longer C310.1
- net BKA_FB: now also R221.2, R222.1; no longer R197.2, R198.1
- net BKA_MODE: now also R220.1; no longer R196.1
- net BKA_SS: now also C315.1; no longer C312.1
- net BKA_SW: now also C313.2; no longer C310.2
- net BKA_VREG5: now also C314.1; no longer C311.1
- net BKC_BOOT: now also C310.1; no longer C307.1
- net BKC_FB: now also R217.2, R218.1; no longer R193.2, R194.1
- net BKC_MODE: now also R216.1; no longer R192.1
- net BKC_SS: now also C312.1; no longer C309.1
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Other:
- note added: "Port modules: TCA9548A U95/U96 (ID EEPROM @0x50 per slot), TCA9555 U97 (PRSNT#)"

Commit message: I/O plate: centre + corner M1.6 frame screws, screwpt variant, plate fixes, module routing, ESD
Parts:
- added C990: 100nF U98 VS, MP62_IO:C_0402_1005Metric, symbol MP62_IO:C
- added D200: TPD4E02B04DQAR (C106794) 0.25 pF ESD - C1 TX1/RX1, MP62_IO:USON-10_2.5x1.0mm_P0.5mm, symbol MP62_IO:ESD4_DQA
- added D201: TPD4E02B04DQAR (C106794) 0.25 pF ESD - C1 TX2/RX2, MP62_IO:USON-10_2.5x1.0mm_P0.5mm, symbol MP62_IO:ESD4_DQA
- added D202: TPD4E05U06DQAR (C138714) 0.5 pF ESD - C1 D+/D-/SB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, MP62_IO:USON-10_2.5x1.0mm_P0.5mm, symbol MP62_IO:ESD4_DQA
- added D203: TPD4E02B04DQAR (C106794) 0.25 pF ESD - C2 TX1/RX1, MP62_IO:USON-10_2.5x1.0mm_P0.5mm, symbol MP62_IO:ESD4_DQA
- added D204: TPD4E02B04DQAR (C106794) 0.25 pF ESD - C2 TX2/RX2, MP62_IO:USON-10_2.5x1.0mm_P0.5mm, symbol MP62_IO:ESD4_DQA
- added D205: TPD4E05U06DQAR (C138714) 0.5 pF ESD - C2 D+/D-/SB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, MP62_IO:USON-10_2.5x1.0mm_P0.5mm, symbol MP62_IO:ESD4_DQA
- added D206: TPD4E02B04DQAR (C106794) 0.25 pF ESD - C3 TX1/RX1, MP62_IO:USON-10_2.5x1.0mm_P0.5mm, symbol MP62_IO:ESD4_DQA
- added D207: TPD4E02B04DQAR (C106794) 0.25 pF ESD - C3 TX2/RX2, MP62_IO:USON-10_2.5x1.0mm_P0.5mm, symbol MP62_IO:ESD4_DQA
- added D208: TPD4E05U06DQAR (C138714) 0.5 pF ESD - C3 D+/D-/SB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, MP62_IO:USON-10_2.5x1.0mm_P0.5mm, symbol MP62_IO:ESD4_DQA
- added D209: TPD4E02B04DQAR (C106794) 0.25 pF ESD - C4 TX1/RX1, MP62_IO:USON-10_2.5x1.0mm_P0.5mm, symbol MP62_IO:ESD4_DQA
- added D210: TPD4E02B04DQAR (C106794) 0.25 pF ESD - C4 TX2/RX2, MP62_IO:USON-10_2.5x1.0mm_P0.5mm, symbol MP62_IO:ESD4_DQA
- added D211: TPD4E05U06DQAR (C138714) 0.5 pF ESD - C4 D+/D-/SB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, MP62_IO:USON-10_2.5x1.0mm_P0.5mm, symbol MP62_IO:ESD4_DQA
- added D212: TPD4E02B04DQAR (C106794) 0.25 pF ESD - C5 TX1/RX1, MP62_IO:USON-10_2.5x1.0mm_P0.5mm, symbol MP62_IO:ESD4_DQA
- added D213: TPD4E02B04DQAR (C106794) 0.25 pF ESD - C5 TX2/RX2, MP62_IO:USON-10_2.5x1.0mm_P0.5mm, symbol MP62_IO:ESD4_DQA
- added D214: TPD4E05U06DQAR (C138714) 0.5 pF ESD - C5 D+/D-/SB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, MP62_IO:USON-10_2.5x1.0mm_P0.5mm, symbol MP62_IO:ESD4_DQA
- added D215: TPD4E02B04DQAR (C106794) 0.25 pF ESD - C6 TX1/RX1, MP62_IO:USON-10_2.5x1.0mm_P0.5mm, symbol MP62_IO:ESD4_DQA
- added D216: TPD4E02B04DQAR (C106794) 0.25 pF ESD - C6 TX2/RX2, MP62_IO:USON-10_2.5x1.0mm_P0.5mm, symbol MP62_IO:ESD4_DQA
- added D217: TPD4E05U06DQAR (C138714) 0.5 pF ESD - C6 D+/D-/SB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, MP62_IO:USON-10_2.5x1.0mm_P0.5mm, symbol MP62_IO:ESD4_DQA
- added D218: TPD4E02B04DQAR (C106794) 0.25 pF ESD - A1 SSTX/SS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, MP62_IO:USON-10_2.5x1.0mm_P0.5mm, symbol MP62_IO:ESD4_DQA
- added D219: TPD4E05U06DQAR (C138714) 0.5 pF ESD - A1 D+/D-, MP62_IO:USON-10_2.5x1.0mm_P0.5mm, symbol MP62_IO:ESD4_DQA
- added D220: TPD4E02B04DQAR (C106794) 0.25 pF ESD - A2 SSTX/SS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, MP62_IO:USON-10_2.5x1.0mm_P0.5mm, symbol MP62_IO:ESD4_DQA
- added D221: TPD4E05U06DQAR (C138714) 0.5 pF ESD - A2 D+/D-, MP62_IO:USON-10_2.5x1.0mm_P0.5mm, symbol MP62_IO:ESD4_DQA
- added D222: TPD4E02B04DQAR (C106794) 0.25 pF ESD - A3 SSTX/SS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, MP62_IO:USON-10_2.5x1.0mm_P0.5mm, symbol MP62_IO:ESD4_DQA
- added D223: TPD4E05U06DQAR (C138714) 0.5 pF ESD - A3 D+/D-, MP62_IO:USON-10_2.5x1.0mm_P0.5mm, symbol MP62_IO:ESD4_DQA
- added D224: TPD4E02B04DQAR (C106794) 0.25 pF ESD - A4 SSTX/SS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, MP62_IO:USON-10_2.5x1.0mm_P0.5mm, symbol MP62_IO:ESD4_DQA
- added D225: TPD4E05U06DQAR (C138714) 0.5 pF ESD - A4 D+/D-, MP62_IO:USON-10_2.5x1.0mm_P0.5mm, symbol MP62_IO:ESD4_DQA
- added D226, D227: TPD4E05U06DQAR (C138714) 0.5 pF ESD - HDMI TMDS D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, MP62_IO:USON-10_2.5x1.0mm_P0.5mm, symbol MP62_IO:ESD4_DQA
- added D228: TPD4E05U06DQAR (C138714) 0.5 pF ESD - HDMI DDC SC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, MP62_IO:USON-10_2.5x1.0mm_P0.5mm, symbol MP62_IO:ESD4_DQA
- added RS90: 1 mOhm 1% 2512 Kelvin shunt (IOB 12 V after U40; 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, MP62_IO:R_2512_6332Metric, symbol MP62_IO:R
- added U98: INA228AIDGSR @0x41 (A0 = VS, A1 = GND), I2C_SYS; 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, MP62_IO:VSSOP-10_3x3mm_P0.5mm, symbol MP62_IO:INA228
- R148: value 0R: Bluetooth 3V3 (card P18) from standby so BT can wake in S3; confirm on M-IOC1 -> 0R DNP alt: BT from standby (no wake path in rev A: hubs S0-only, no S3) - Aidan 2026-10-02 / ICD O-3; now not fitted; now left out of the parts list
- R149: value 0R DNP alt: BT from S0 3V3 -> 0R: Bluetooth 3V3 (card P18) from S0 3V3 (default, Aidan 2026-10-02 / ICD O-3); now fitted; now in the parts list
Connections:
- net +12V_IOB: now also RS90.2, U98.2 (IN-), U98.3 (VBUS); no longer U40.6 (OUT)
- net 3V3: now also JM1.46 (3V3_MOD), JM10.46 (3V3_MOD), JM11.46 (3V3_MOD), JM2.46 (3V3_MOD), JM3.46 (3V3_MOD), JM4.46 (3V3_MOD), JM5.46 (3V3_MOD), JM6.46 (3V3_MOD), JM7.46 (3V3_MOD), JM8.46 (3V3_MOD), JM9.46 (3V3_MOD); no longer JM1.43 (3V3_MOD), JM10.43 (3V3_MOD), JM11.43 (3V3_MOD), JM2.43 (3V3_MOD), JM3.43 (3V3_MOD), JM4.43 (3V3_MOD), JM5.43 (3V3_MOD), JM6.43 (3V3_MOD), JM7.43 (3V3_MOD), JM8.43 (3V3_MOD), JM9.43 (3V3_MOD)
- net 3V3_SB: now also C990.1, U98.4 (VS), U98.9 (A0)
- net A1_SS_RX_N: now also JM7.27 (HS3_A), D218.5 (IO4); no longer JM7.25 (HS1_N)
- net A1_SS_RX_P: now also JM7.29 (HS3_B), D218.4 (IO3); no longer JM7.23 (HS1_P)
- net A1_SS_TX_N: now also JM7.33 (HS0_A), D218.2 (IO2); no longer JM7.19 (HS0_N)
- net A1_SS_TX_P: now also JM7.35 (HS0_B), D218.1 (IO1); no longer JM7.17 (HS0_P)
- net A1_USB2_DN: now also JM7.18 (LS_B2), D219.2 (IO2); no longer JM7.31 (USB2_DN)
- net A1_USB2_DP: now also JM7.16 (LS_B1), D219.1 (IO1); no longer JM7.29 (USB2_DP)
- net A2_SS_RX_N: now also JM8.27 (HS3_A), D220.5 (IO4); no longer JM8.25 (HS1_N)
- net A2_SS_RX_P: now also JM8.29 (HS3_B), D220.4 (IO3); no longer JM8.23 (HS1_P)
- net A2_SS_TX_N: now also JM8.33 (HS0_A), D220.2 (IO2); no longer JM8.19 (HS0_N)
- net A2_SS_TX_P: now also JM8.35 (HS0_B), D220.1 (IO1); no longer JM8.17 (HS0_P)
- net A2_USB2_DN: now also JM8.18 (LS_B2), D221.2 (IO2); no longer JM8.31 (USB2_DN)
- net A2_USB2_DP: now also JM8.16 (LS_B1), D221.1 (IO1); no longer JM8.29 (USB2_DP)
- net A3_SS_RX_N: now also JM9.27 (HS3_A), D222.5 (IO4); no longer JM9.25 (HS1_N)
- net A3_SS_RX_P: now also JM9.29 (HS3_B), D222.4 (IO3); no longer JM9.23 (HS1_P)
- net A3_SS_TX_N: now also JM9.33 (HS0_A), D222.2 (IO2); no longer JM9.19 (HS0_N)
- net A3_SS_TX_P: now also JM9.35 (HS0_B), D222.1 (IO1); no longer JM9.17 (HS0_P)
- net A3_USB2_DN: now also JM9.18 (LS_B2), D223.2 (IO2); no longer JM9.31 (USB2_DN)
- net A3_USB2_DP: now also JM9.16 (LS_B1), D223.1 (IO1); no longer JM9.29 (USB2_DP)
- net A4_SS_RX_N: now also JM10.27 (HS3_A), D224.5 (IO4); no longer JM10.25 (HS1_N)
- net A4_SS_RX_P: now also JM10.29 (HS3_B), D224.4 (IO3); no longer JM10.23 (HS1_P)
- net A4_SS_TX_N: now also JM10.33 (HS0_A), D224.2 (IO2); no longer JM10.19 (HS0_N)
- net A4_SS_TX_P: now also JM10.35 (HS0_B), D224.1 (IO1); no longer JM10.17 (HS0_P)
- net A4_USB2_DN: now also JM10.18 (LS_B2), D225.2 (IO2); no longer JM10.31 (USB2_DN)
- net A4_USB2_DP: now also JM10.16 (LS_B1), D225.1 (IO1); no longer JM10.29 (USB2_DP)
- net C1_CC1: now also JM1.21 (LS_A1); no longer JM1.35 (CC1)
- net C1_CC2: now also JM1.16 (LS_B1); no longer JM1.37 (CC2)
- net C1_SBU1: now also JM1.23 (LS_A2), D202.4 (IO3); no longer JM1.30 (SBU1)
- net C1_SBU2: now also JM1.18 (LS_B2), D202.5 (IO4); no longer JM1.32 (SBU2)
- net C1_SS_RX1_N: now also JM1.34 (HS1_A), D200.5 (IO4); no longer JM1.25 (HS1_N)
- net C1_SS_RX1_P: now also JM1.36 (HS1_B), D200.4 (IO3); no longer JM1.23 (HS1_P)
- net C1_SS_RX2_N: now also JM1.29 (HS3_B), D201.5 (IO4); no longer JM1.26 (HS3_N)
- net C1_SS_RX2_P: now also JM1.27 (HS3_A), D201.4 (IO3); no longer JM1.24 (HS3_P)
- net C1_SS_TX1_N: now also JM1.33 (HS0_A), D200.2 (IO2); no longer JM1.19 (HS0_N)
- net C1_SS_TX1_P: now also JM1.35 (HS0_B), D200.1 (IO1); no longer JM1.17 (HS0_P)
- net C1_SS_TX2_N: now also JM1.30 (HS2_B), D201.2 (IO2); no longer JM1.20 (HS2_N)
- net C1_SS_TX2_P: now also JM1.28 (HS2_A), D201.1 (IO1); no longer JM1.18 (HS2_P)
- net C1_USB2_DN: now also JM1.17 (USB2_B), D202.2 (IO2); no longer JM1.31 (USB2_DN)
- net C1_USB2_DP: now also JM1.15 (USB2_A), D202.1 (IO1); no longer JM1.29 (USB2_DP)
- net C2_CC1: now also JM2.21 (LS_A1); no longer JM2.35 (CC1)
- net C2_CC2: now also JM2.16 (LS_B1); no longer JM2.37 (CC2)
- net C2_SBU1: now also JM2.23 (LS_A2), D205.4 (IO3); no longer JM2.30 (SBU1)
- net C2_SBU2: now also JM2.18 (LS_B2), D205.5 (IO4); no longer JM2.32 (SBU2)
- net C2_SS_RX1_N: now also JM2.34 (HS1_A), D203.5 (IO4); no longer JM2.25 (HS1_N)
- net C2_SS_RX1_P: now also JM2.36 (HS1_B), D203.4 (IO3); no longer JM2.23 (HS1_P)
- net C2_SS_RX2_N: now also JM2.29 (HS3_B), D204.5 (IO4); no longer JM2.26 (HS3_N)
- net C2_SS_RX2_P: now also JM2.27 (HS3_A), D204.4 (IO3); no longer JM2.24 (HS3_P)
- net C2_SS_TX1_N: now also JM2.33 (HS0_A), D203.2 (IO2); no longer JM2.19 (HS0_N)
- net C2_SS_TX1_P: now also JM2.35 (HS0_B), D203.1 (IO1); no longer JM2.17 (HS0_P)
- net C2_SS_TX2_N: now also JM2.30 (HS2_B), D204.2 (IO2); no longer JM2.20 (HS2_N)
- net C2_SS_TX2_P: now also JM2.28 (HS2_A), D204.1 (IO1); no longer JM2.18 (HS2_P)
- net C2_USB2_DN: now also JM2.17 (USB2_B), D205.2 (IO2); no longer JM2.31 (USB2_DN)
- net C2_USB2_DP: now also JM2.15 (USB2_A), D205.1 (IO1); no longer JM2.29 (USB2_DP)
- net C3_CC1: now also JM3.21 (LS_A1); no longer JM3.35 (CC1)
- net C3_CC2: now also JM3.16 (LS_B1); no longer JM3.37 (CC2)
- net C3_SBU1: now also JM3.23 (LS_A2), D208.4 (IO3); no longer JM3.30 (SBU1)
- net C3_SBU2: now also JM3.18 (LS_B2), D208.5 (IO4); no longer JM3.32 (SBU2)
- net C3_SS_RX1_N: now also JM3.34 (HS1_A), D206.5 (IO4); no longer JM3.25 (HS1_N)
- net C3_SS_RX1_P: now also JM3.36 (HS1_B), D206.4 (IO3); no longer JM3.23 (HS1_P)
- net C3_SS_RX2_N: now also JM3.29 (HS3_B), D207.5 (IO4); no longer JM3.26 (HS3_N)
- net C3_SS_RX2_P: now also JM3.27 (HS3_A), D207.4 (IO3); no longer JM3.24 (HS3_P)
- net C3_SS_TX1_N: now also JM3.33 (HS0_A), D206.2 (IO2); no longer JM3.19 (HS0_N)
- net C3_SS_TX1_P: now also JM3.35 (HS0_B), D206.1 (IO1); no longer JM3.17 (HS0_P)
- net C3_SS_TX2_N: now also JM3.30 (HS2_B), D207.2 (IO2); no longer JM3.20 (HS2_N)
- net C3_SS_TX2_P: now also JM3.28 (HS2_A), D207.1 (IO1); no longer JM3.18 (HS2_P)
- net C3_USB2_DN: now also JM3.17 (USB2_B), D208.2 (IO2); no longer JM3.31 (USB2_DN)
- net C3_USB2_DP: now also JM3.15 (USB2_A), D208.1 (IO1); no longer JM3.29 (USB2_DP)
- net C4_CC1: now also JM4.21 (LS_A1); no longer JM4.35 (CC1)
- net C4_CC2: now also JM4.16 (LS_B1); no longer JM4.37 (CC2)
- net C4_SBU1: now also JM4.23 (LS_A2), D211.4 (IO3); no longer JM4.30 (SBU1)
- net C4_SBU2: now also JM4.18 (LS_B2), D211.5 (IO4); no longer JM4.32 (SBU2)
- net C4_SS_RX1_N: now also JM4.34 (HS1_A), D209.5 (IO4); no longer JM4.25 (HS1_N)
- net C4_SS_RX1_P: now also JM4.36 (HS1_B), D209.4 (IO3); no longer JM4.23 (HS1_P)
- net C4_SS_RX2_N: now also JM4.29 (HS3_B), D210.5 (IO4); no longer JM4.26 (HS3_N)
- net C4_SS_RX2_P: now also JM4.27 (HS3_A), D210.4 (IO3); no longer JM4.24 (HS3_P)
- net C4_SS_TX1_N: now also JM4.33 (HS0_A), D209.2 (IO2); no longer JM4.19 (HS0_N)
- net C4_SS_TX1_P: now also JM4.35 (HS0_B), D209.1 (IO1); no longer JM4.17 (HS0_P)
- net C4_SS_TX2_N: now also JM4.30 (HS2_B), D210.2 (IO2); no longer JM4.20 (HS2_N)
- net C4_SS_TX2_P: now also JM4.28 (HS2_A), D210.1 (IO1); no longer JM4.18 (HS2_P)
- net C4_USB2_DN: now also JM4.17 (USB2_B), D211.2 (IO2); no longer JM4.31 (USB2_DN)
- net C4_USB2_DP: now also JM4.15 (USB2_A), D211.1 (IO1); no longer JM4.29 (USB2_DP)
- net C5_CC1: now also JM5.21 (LS_A1); no longer JM5.35 (CC1)
- net C5_CC2: now also JM5.16 (LS_B1); no longer JM5.37 (CC2)
- net C5_SBU1: now also JM5.23 (LS_A2), D214.4 (IO3); no longer JM5.30 (SBU1)
- net C5_SBU2: now also JM5.18 (LS_B2), D214.5 (IO4); no longer JM5.32 (SBU2)
- net C5_SS_RX1_N: now also JM5.34 (HS1_A), D212.5 (IO4); no longer JM5.25 (HS1_N)
- net C5_SS_RX1_P: now also JM5.36 (HS1_B), D212.4 (IO3); no longer JM5.23 (HS1_P)
- net C5_SS_RX2_N: now also JM5.29 (HS3_B), D213.5 (IO4); no longer JM5.26 (HS3_N)
- net C5_SS_RX2_P: now also JM5.27 (HS3_A), D213.4 (IO3); no longer JM5.24 (HS3_P)
- net C5_SS_TX1_N: now also JM5.33 (HS0_A), D212.2 (IO2); no longer JM5.19 (HS0_N)
- net C5_SS_TX1_P: now also JM5.35 (HS0_B), D212.1 (IO1); no longer JM5.17 (HS0_P)
- net C5_SS_TX2_N: now also JM5.30 (HS2_B), D213.2 (IO2); no longer JM5.20 (HS2_N)
- net C5_SS_TX2_P: now also JM5.28 (HS2_A), D213.1 (IO1); no longer JM5.18 (HS2_P)
- net C5_USB2_DN: now also JM5.17 (USB2_B), D214.2 (IO2); no longer JM5.31 (USB2_DN)
- new net +12V_EFUSE_OUT: RS90.1, U40.6 (OUT), U98.1 (IN+)
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
Commit message: USB-C flex module routed (HYCW417, 0 DRC, matched pairs), 3-mil min on flexes, two flex panels, CH334F + ASM1182e QFN-48 footprints
Parts:
- removed U32: CH334R H1b <- H1a port 4, MP62_IO:MP62_WCH_CH334R_QFN-24_4x4_P0.5_PLACEHOLDER, symbol MP62_IO:CH334R
- removed U33: CH334R H2 <- IOB-LINK USB2 (BP spare), MP62_IO:MP62_WCH_CH334R_QFN-24_4x4_P0.5_PLACEHOLDER, symbol MP62_IO:CH334R
- removed U34: CH334R H1a <- HS1 USB2 (CB PCH port), MP62_IO:MP62_WCH_CH334R_QFN-24_4x4_P0.5_PLACEHOLDER, symbol MP62_IO:CH334R
- removed U35: CH334R H3 <- H2 port 4 (A4 + AirPort Bluetooth + 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, MP62_IO:MP62_WCH_CH334R_QFN-24_4x4_P0.5_PLACEHOLDER, symbol MP62_IO:CH334R
- added U32: CH334F H1b <- H1a port 4, MP62_IO:MP62_WCH_CH334F_QFN-24-1EP_4x4_P0.5_EP2.8, symbol MP62_IO:CH334F
- added U33: CH334F H2 <- IOB-LINK USB2 (BP spare), MP62_IO:MP62_WCH_CH334F_QFN-24-1EP_4x4_P0.5_EP2.8, symbol MP62_IO:CH334F
- added U34: CH334F H1a <- HS1 USB2 (CB PCH port), MP62_IO:MP62_WCH_CH334F_QFN-24-1EP_4x4_P0.5_EP2.8, symbol MP62_IO:CH334F
- added U35: CH334F H3 <- H2 port 4 (A4 + AirPort Bluetooth + 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, MP62_IO:MP62_WCH_CH334F_QFN-24-1EP_4x4_P0.5_EP2.8, symbol MP62_IO:CH334F
- U91: footprint MP62_IO:MP62_ASMedia_ASM1182e_QFN-64_9x9_P0.5_PLACEHOLDER -> MP62_IO:MP62_ASMedia_ASM1182e_QFN-48-1EP_7x7_P0.5_EP5.4
Connections:
- net 5V_A: now also U32.5 (V5), U33.5 (V5), U34.5 (V5), U35.5 (V5)
- net A1_USB2_DN: now also U33.10 (DM1)
- net A1_USB2_DP: now also U33.9 (DP1)
- net A2_USB2_DN: now also U33.12 (DM2)
- net A2_USB2_DP: now also U33.11 (DP2)
- net A3_USB2_DN: now also U33.14 (DM3)
- net A3_USB2_DP: now also U33.13 (DP3)
- net A4_USB2_DN: now also U35.10 (DM1)
- net A4_USB2_DP: now also U35.9 (DP1)
- net AUD_USB2_DN: now also U32.16 (DM4)
- net AUD_USB2_DP: now also U32.15 (DP4)
- net BT_USB2_DN: now also U35.12 (DM2)
- net BT_USB2_DP: now also U35.11 (DP2)
- net C1_USB2_DN: now also U34.10 (DM1)
- net C1_USB2_DP: now also U34.9 (DP1)
- net C2_USB2_DN: now also U34.12 (DM2)
- net C2_USB2_DP: now also U34.11 (DP2)
- net C3_USB2_DN: now also U34.14 (DM3)
- net C3_USB2_DP: now also U34.13 (DP3)
- net C4_USB2_DN: now also U32.10 (DM1)
- net C4_USB2_DP: now also U32.9 (DP1)
- net C5_USB2_DN: now also U32.12 (DM2)
- net C5_USB2_DP: now also U32.11 (DP2)
- net C6_USB2_DN: now also U32.14 (DM3)
- net C6_USB2_DP: now also U32.13 (DP3)
- net GND: now also U32.17 (EP_GND), U32.8 (GND), U33.17 (EP_GND), U33.8 (GND), U34.17 (EP_GND), U34.8 (GND), U35.17 (EP_GND), U35.8 (GND)
- net H1B_USB2_DN: now also U32.2 (UDM), U34.16 (DM4)
- net H1B_USB2_DP: now also U32.1 (UDP), U34.15 (DP4)
- net H3_USB2_DN: now also U33.16 (DM4), U35.2 (UDM)
- net H3_USB2_DP: now also U33.15 (DP4), U35.1 (UDP)
- net U32_V33: now also U32.6 (V33), U32.7 (RESET#)
- net U32_XI: now also U32.3 (XI)
- net U32_XO: now also U32.4 (XO)
- net U33_V33: now also U33.6 (V33), U33.7 (RESET#)
- net U33_XI: now also U33.3 (XI)
- net U33_XO: now also U33.4 (XO)
- net U34_V33: now also U34.6 (V33), U34.7 (RESET#)
- net U34_XI: now also U34.3 (XI)
- net U34_XO: now also U34.4 (XO)
- net U35_V33: now also U35.6 (V33), U35.7 (RESET#)
- net U35_XI: now also U35.3 (XI)
- net U35_XO: now also U35.4 (XO)
- net USB2_HS1_DN: now also U34.2 (UDM)
- net USB2_HS1_DP: now also U34.1 (UDP)
- net USB2_LINK_DN: now also U33.2 (UDM)
- net USB2_LINK_DP: now also U33.1 (UDP)
Other:
- note added: "USB2 hubs CH334F (H1a U34, H1b U32, H2 U33, H3 U35)"
- note removed: "USB2 hubs CH334R (H1a U34, H1b U32, H2 U33, H3 U35)"
