File: kicad/macpro62-io-board/macpro62-io-board.kicad_sch (KiCad schematic)
At the start: 510 parts, among them J1 IOB-HS1 MCIO 124 RA <- CB J3, J2 DISPLAY-LINK MCIO 74 RA <- Fa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, J25 Non-magnetic vertical RJ45 (E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, J26 Non-magnetic vertical RJ45 (E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, J28 Stock audio module connector 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, J29 Speaker 2P JST SH vertical (s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, J3 Stock PSU DC-out 12P (PROVISI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, J30 OPTIONAL 2P: stock I/O-wall b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, J31 I/O-wall flex ZIF 14P 0.5 (st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, J4 Stock PSU signal 6P (PROVISIO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, J5 Micro-Fit 2x4 -> BP J2 (1-2 1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, J6 IOB-LINK GH15 vertical <- BP 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, J7 CONN_C fan + AirPort (stock p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, J8 Fan-assembly antenna coax (st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, J9 Optional antenna pass-through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, Q90 MMBT3904 remote diode (or omi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, SW1 Power button PTS810 on the IO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, SW2 DIAG button TL3342 (back side), T1 JASN V24P05S 2.5G magnetics (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, T2 JASN V24P05S 2.5G magnetics (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, U1 TPS65994AD PD #1 (C1, C2), U11 TUSB1046A-DCI C1 mux/redriver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, U12 TUSB1046A-DCI C2 mux/redriver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, U13 TUSB1046A-DCI C3 mux/redriver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, U14 TUSB1046A-DCI C4 mux/redriver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, U15 TUSB1046A-DCI C5 mux/redriver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, U16 TUSB1046A-DCI C6 mux/redriver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, U2 TPS65994AD PD #2 (C3, C4), U21 TUSB1002A A1 redriver, U22 TUSB1002A A2 redriver, U23 TUSB1002A A3 redriver, U24 TUSB1002A A4 redriver, U25 SY6280AAC / TPS2553 1.5 A swi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, U26 SY6280AAC / TPS2553 1.5 A swi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, U27 SY6280AAC / TPS2553 1.5 A swi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, U28 SY6280AAC / TPS2553 1.5 A swi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, U3 TPS65994AD PD #3 (C5, C6), U30 DRV5032FB (OD, 5 Hz low power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, U31 DRV5032FB (OD, 5 Hz low power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, U32 CH334F H1b <- H1a port 4, U33 CH334F H2 <- IOB-LINK USB2 (B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, U34 CH334F H1a <- HS1 USB2 (CB PC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, U35 CH334F H3 <- H2 port 4 (A4 + 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, U4 W25Q80DV class 8 Mbit (PD #1 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, U40 TPS259824ONRGER eFuse 12 V (I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, U41 TPS56C215RNNR 5V_C buck 12 A, U42 TPS56C215RNNR 5V_A buck 12 A, U43 TLV62585DRL 3V3 3 A from 5V_A, U50 Intel i226-V 2.5GbE #1 (HS1 k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, U51 i226 #1 NVM 2 Mbit+ SPI flash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, U52 Intel i226-V 2.5GbE #2 (HS1 k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, U53 i226 #2 NVM 2 Mbit+ SPI flash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, U6 W25Q80DV class 8 Mbit (PD #2 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, U60 TDP158RSBR HDMI retimer, U61 TLV75511PDBV 1.1 V LDO (TDP15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, U7 W25Q80DV class 8 Mbit (PD #3 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, U70 CM108B USB audio codec (UAC1), U71 PAM8302AAS 2.5 W mono class-D, U80 TLC59116IPWR @0x60 (A3..A0 = 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, U81 LIS2DH12TR @0x18 (optional ro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, U82 BL24C64A-SFRC IOB ID EEPROM @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, U83 TCA9517DGKR I2C buffer: I2C_S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, U84 74LVC1G07 PD_INT_N -> IOB_INT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, U90 EMC2101 fan controller (SMBus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, U91 ASM1182e PCIe Gen2 switch: up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, U92 3V3 WLAN load switch (TPS2291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, U95 TCA9548APWR @0x70: ch0-5 C1-C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, U96 TCA9548APWR @0x71: ch0-1 A3-A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, U97 TCA9555PWR @0x27 on U96 ch3 (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, U98 INA228AIDGSR @0x41 (A0 = VS, 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, Y1 12MHz 3225 +/-20ppm, Y2 12MHz 3225 +/-20ppm, Y3 12MHz 3225 +/-20ppm, Y4 25MHz 3225 +/-30ppm (i226 #1), Y5 12MHz 3225 (CM108B), Y6 25MHz 3225 +/-30ppm (i226 #2), Y7 12MHz 3225 +/-20ppm, Y8 25MHz 3225 (ASM1182e, per dat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

Commit message: Plate test-print fixes (corners +1mm Y, C2 post -1mm, C1 removed); USB-A/HDMI hand fan-out 0 skew; real DF40 + HDMI footprints
Parts:
- JM1, JM10, JM11, JM2, JM3, JM4, JM5, JM6, JM7, JM8, JM9: footprint MP62_IO:MP62_Hirose_DF40C-50DS-0.4V_PLACEHOLDER -> MP62_IO:MP62_Hirose_DF40C-50DS-0.4V
Connections:
- net HDMI_HPD: now also JM11.22 (SPARE_B1); no longer JM11.16 (LS_B1)
- net HDMI_SCL: now also JM11.16 (LS_B1); no longer JM11.18 (LS_B2)
- net HDMI_SDA: now also JM11.18 (LS_B2); no longer JM11.23 (LS_A2)
- net TMDS_CK_N: now also JM11.15 (USB2_A); no longer JM11.27 (HS3_A)
- net TMDS_CK_P: now also JM11.17 (USB2_B); no longer JM11.29 (HS3_B)
- net TMDS_D0_N: now also JM11.21 (LS_A1); no longer JM11.28 (HS2_A)
- net TMDS_D0_P: now also JM11.23 (LS_A2); no longer JM11.30 (HS2_B)
- net TMDS_D1_N: now also JM11.27 (HS3_A); no longer JM11.33 (HS0_A)
- net TMDS_D1_P: now also JM11.29 (HS3_B); no longer JM11.35 (HS0_B)
- net TMDS_D2_N: now also JM11.33 (HS0_A); no longer JM11.34 (HS1_A)
- net TMDS_D2_P: now also JM11.35 (HS0_B); no longer JM11.36 (HS1_B)
